Commit message: add camera collision area, closes #19

File: mogi_chess_gazebo/urdf/camera.xacro (robot description, xacro)
@@ -3,5 +3,5 @@
   <!-- Camera -->
   <joint type="fixed" name="camera_joint">
-    <origin xyz="-0.3 0.3 0.6" rpy="0 1.1 0"/>
+    <origin xyz="-0.3 0.3 0.55" rpy="0 1.05 0"/>
     <child link="camera_link"/>
     <parent link="world"/>
@@ -20,7 +20,7 @@
     </inertial>
     <collision name='collision'>
-      <origin xyz="0 0 0" rpy="0 0 0"/>
+      <origin xyz="0 0 0" rpy="0 1.5707 0"/>
       <geometry>
-        <box size=".05 .05 .05"/>
+        <cylinder length="0.05" radius="0.1"/>
       </geometry>
     </collision>
